Commit message: Checkpoint: mecanum 4-wheel AMR - Nav2 narrow-passage tuning + RF2O fixes
Snapshot of the full mecanum-drivetrain platform before starting the
2WD + caster drivetrain transition. Covers this session's accumulated
work: mecanum wheel contactMaterial/friction physics, narrow-passage
costmap inflation and DWB critic tuning, behavior_server plugin/frame
corrections, velocity_smoother wiring, controller_server odom_topic
fix, and the RF2O publish-gating submodule fix (see
src/rf2o_laser_odometry's own history for that commit).

Co-Authored-By: Claude Sonnet 5 <noreply@anthropic.com>

File: src/amr_description/urdf/mech/wheel.urdf.xacro (robot description, xacro)
@@ -7,5 +7,9 @@
   <xacro:property name="wheel_xoff" value="0.08" />
   <xacro:property name="wheel_yoff" value="-0.01" />
-  <xacro:macro name="wheel" params="prefix side x_reflect y_reflect">
+  <!-- contact_material: "wheel_pos_45" for FL+RR (roller angle +45 deg),
+                          "wheel_neg_45" for FR+RL (roller angle -45 deg).
+       Injected as a Webots contactMaterial field on each wheel Solid
+       by fix_proto.py post-processing. No effect in Gazebo/RViz. -->
+  <xacro:macro name="wheel" params="prefix side x_reflect y_reflect contact_material">
     <link name="${prefix}${side}_wheel_link">
       <visual>
@@ -38,10 +42,12 @@
       <child link="${prefix}${side}_wheel_link"/>
       <origin xyz="${x_reflect*wheel_xoff} ${y_reflect*(wheel_separation/2+wheel_yoff)} ${-wheel_radius}" rpy="0 0 0"/>
-      <dynamics damping="0.1" friction="0.05"/>
+      <dynamics damping="0.01" friction="0.01"/>
+      <limit effort="30.0" velocity="15.0"/>
     </joint>
+    <!-- Gazebo / ROS 2 control surface properties -->
     <gazebo reference="${prefix}${side}_wheel_link">
-      <mu1>0.8</mu1>      <!-- High friction along the rolling direction -->
-      <mu2>0.8</mu2>      <!-- High friction along the sliding axis -->
-      <fdir1>1 0 0</fdir1> <!-- Specifies the primary rolling direction -->
+      <mu1>0.8</mu1>
+      <mu2>0.8</mu2>
+      <fdir1>1 0 0</fdir1>
       <surface>
         <friction>

File: src/amr_description/urdf/robots/amr.urdf.xacro (robot description, xacro)
@@ -16,20 +16,24 @@
       side="front_left"
       x_reflect="1"
-      y_reflect="1"/>
+      y_reflect="1"
+      contact_material="wheel_pos_45"/>
     <xacro:wheel
       prefix="$(arg prefix)"
       side="front_right"
       x_reflect="1"
-      y_reflect="-1"/>
+      y_reflect="-1"
+      contact_material="wheel_neg_45"/>
     <xacro:wheel
       prefix="$(arg prefix)"
       side="rear_left"
       x_reflect="-1"
-      y_reflect="1"/>
+      y_reflect="1"
+      contact_material="wheel_neg_45"/>
     <xacro:wheel
       prefix="$(arg prefix)"
       side="rear_right"
       x_reflect="-1"
-      y_reflect="-1"/>
+      y_reflect="-1"
+      contact_material="wheel_pos_45"/>
     <xacro:camera
       prefix="$(arg prefix)"
