Commit message: Checkpoint: rmp_bot-based 2WD + caster transition (pre-TurtleBot3 pivot)
Snapshot of the 2-wheel differential drive + passive caster platform
(chassis/wheel/caster geometry and mass from
github.com/ravithakur-projects/ROS-Three-Wheeled-Robot-Navigation-Project,
diff_drive_controller wiring, AMCL DifferentialMotionModel, corrected
wheel/caster mesh transforms and collision primitives, lidar mount height
fix) before starting a full migration to the standard ROBOTIS TurtleBot3
Burger + webots_ros2_turtlebot packages.

Co-Authored-By: Claude Sonnet 5 <noreply@anthropic.com>

File: src/amr_description/urdf/control/ros2_control.urdf.xacro (robot description, xacro)
@@ -11,5 +11,5 @@
         </xacro:if>
       </hardware>
-      <joint name="${prefix}front_left_wheel_joint">
+      <joint name="${prefix}left_wheel_joint">
         <command_interface name="velocity">
           <param name="min">-50.0</param>
@@ -19,21 +19,5 @@
         <state_interface name="velocity"/>
       </joint>
-      <joint name="${prefix}front_right_wheel_joint">
-        <command_interface name="velocity">
-          <param name="min">-50.0</param>
-          <param name="max">50.0</param>
-        </command_interface>
-        <state_interface name="position"/>
-        <state_interface name="velocity"/>
-      </joint>
-      <joint name="${prefix}rear_left_wheel_joint">
-        <command_interface name="velocity">
-          <param name="min">-50.0</param>
-          <param name="max">50.0</param>
-        </command_interface>
-        <state_interface name="position"/>
-        <state_interface name="velocity"/>
-      </joint>
-      <joint name="${prefix}rear_right_wheel_joint">
+      <joint name="${prefix}right_wheel_joint">
         <command_interface name="velocity">
           <param name="min">-50.0</param>

File: src/amr_description/urdf/control/velocity_control.urdf.xacro (robot description, xacro)
@@ -7,5 +7,5 @@
                     filename="gz-sim-velocity-control-system"
                     name="gz::sim::systems::VelocityControl">
-                    <topic>mecanum_drive_controller/cmd_vel</topic>
+                    <topic>diff_drive_controller/cmd_vel</topic>
                     <initial_linear>0 0 0</initial_linear>
                     <initial_angular>0 0 0</initial_angular>

File: src/amr_description/urdf/mech/base.urdf.xacro (robot description, xacro)
@@ -1,19 +1,49 @@
 <?xml version="1.0"?>
 <robot xmlns:xacro="http://www.ros.org/wiki/xacro">
-<xacro:property name="wheel_width" value="0.0304" />
+<!-- wheel_width/wheel_radius here are for the base_z_offset computation
+     only - the authoritative per-wheel values (now measured off rmp_bot's
+     r_wheel_1.stl bounding box: radius 32.5mm, width 25mm) live in
+     wheel.urdf.xacro. Duplicated rather than xacro:included across files
+     to avoid a circular include; kept numerically identical to that file
+     by convention, same as the original mecanum version of this file did. -->
+<xacro:property name="wheel_width" value="0.025" />
 <xacro:property name="wheel_radius" value="0.0325" />
-<xacro:property name="base_mass" value="4.6" />
-<!-- Collision/inertial box aligned to the physical chassis body of the
-     MicroROS-V2 / ROSMASTER-X3: 280mm x 220mm x 150mm (length x width x height).
-     The chassis sits on the wheel axle plane; base_link origin is at ground level
-     so the chassis body centroid is offset +Z by wheel_radius + chassis_height/2.
-     Previous values (0.2924 x 0.1650 x 0.2446) were STL full-extent including
-     the lidar mast tower, making the collision box far taller than the chassis body
-     and causing BackUp to falsely detect floor collisions during recovery. -->
-<xacro:property name="chassis_length" value="0.28"/>
-<xacro:property name="chassis_width"  value="0.22"/>
-<xacro:property name="chassis_height" value="0.15"/>
+<!-- rmp_bot's base_link inertial mass (github.com/ravithakur-projects/
+     ROS-Three-Wheeled-Robot-Navigation-Project) - chassis body only, not
+     including the wheels/caster/sensor payload, matching this project's
+     existing convention of a chassis-only base_mass with sensors/wheels
+     mass-modeled as separate links. -->
+<xacro:property name="base_mass" value="7.21" />
+<!-- Collision/inertial box sized from rmp_bot's base_link.stl bounding box
+     (200mm x 170mm x 110mm, length x width x height - measured directly off
+     the mesh, not the STL's lidar/lidar-mast-inclusive fallback that caused
+     issues on the old chassis). base_link origin is at ground level (matches
+     rmp_bot's own convention: its wheel joints place the axle at
+     z=+wheel_radius above base_link, i.e. base_link = ground plane), so the
+     chassis body centroid is offset +Z by chassis_height/2 only - no
+     wheel_radius term needed here since rmp_bot's base_link origin is
+     already at ground level, unlike the old chassis which had it offset. -->
+<xacro:property name="chassis_length" value="0.20"/>
+<xacro:property name="chassis_width"  value="0.17"/>
+<xacro:property name="chassis_height" value="0.11"/>
 <xacro:property name="base_x_offset" value="0.0"/>
-<xacro:property name="base_z_offset" value="${wheel_radius + chassis_height / 2.0}"/>
+<xacro:property name="base_z_offset" value="${chassis_height / 2.0}"/>
+<!-- Passive rear caster: uses rmp_bot's real caster_1.stl mesh directly for
+     both visual AND collision (not a primitive approximation) - matching
+     their own xacro exactly, which also collides against the raw mesh
+     rather than a sphere/box stand-in. Mass and inertia are rmp_bot's own
+     measured caster_1 inertial values, not a derived formula. -->
+<xacro:property name="caster_mass" value="0.04549"/>
+<xacro:property name="caster_ixx" value="3e-06"/>
+<xacro:property name="caster_iyy" value="3e-06"/>
+<xacro:property name="caster_izz" value="7e-06"/>
+<!-- rmp_bot's exact joint (Rigid5) and visual/collision origin values for
+     caster_1, reproduced as-is rather than re-derived: joint places the
+     link at xyz="0.1 0.0 0.0075" relative to base_link; the mesh's own
+     visual/collision origin is the exact negation, "-0.1 -0.0 -0.0075"
+     (same raw-vertices-in-base_link-frame convention their wheel meshes
+     use - see wheel.urdf.xacro's comment on this). -->
+<xacro:property name="caster_x_offset" value="0.1"/>
+<xacro:property name="caster_z_offset" value="0.0075"/>
 <xacro:macro name="base" params="prefix">
   <xacro:unless value="$(arg use_webots)">
@@ -28,5 +58,8 @@
     <visual>
         <geometry>
-            <mesh filename="package://amr_description/meshes/chassis.stl"/>
+            <!-- rmp_bot's STLs are raw CAD exports in millimeters (matches
+                 the scale="0.001 0.001 0.001" its own xacro applies) -
+                 required here or the chassis renders 1000x too large. -->
+            <mesh filename="package://amr_description/meshes/chassis.stl" scale="0.001 0.001 0.001"/>
         </geometry>
         <material name="green">
@@ -59,4 +92,63 @@
     </visual>
   </gazebo>
+  <link name="${prefix}caster_wheel_link">
+    <visual>
+      <origin xyz="${-caster_x_offset} 0 ${-caster_z_offset}" rpy="0 0 0"/>
+      <geometry>
+        <mesh filename="package://amr_description/meshes/caster_1.stl" scale="0.001 0.001 0.001"/>
+      </geometry>
+      <material name="dark_gray">
+        <color rgba="0.2 0.2 0.2 1.0"/>
+      </material>
+    </visual>
+    <!-- Collision stays a primitive, NOT the scaled mesh used for visual:
+         urdf2webots (this project's R2025a target) prints "BoundingObjects
+         (collisions tags) cannot be scaled in version R2023b and above!"
+         for a scaled mesh boundingObject and falls back to reusing the
+         mesh's UNSCALED (raw millimeter) geometry for collision - a ~1000x
+         oversized collision shape, confirmed by reading the generated
+         proto directly. A cylinder matching the disc's real footprint
+         (40mm diameter, 7.5mm tall) is the correct fix, consistent with
+         how this project already handles collision everywhere else
+         (chassis: mesh visual + box collision; wheels: mesh visual +
+         cylinder collision) - not a new inconsistency. -->
+    <!-- z=-length/2, not 0: the joint's mount point (caster_z_offset) is
+         the disc's TOP surface, not its center (derived from rmp_bot's own
+         mesh - raw vertices span z=[0,0.0075] and the joint sits at the
+         mesh's top edge). A cylinder centered at the link's own origin
+         would float with its bottom 3.75mm above the ground; shifting down
+         by half the height puts the bottom exactly at ground level,
+         matching the real mesh's [0, 0.0075] span. -->
+    <collision>
+      <origin xyz="0 0 -0.00375" rpy="0 0 0"/>
+      <geometry>
+        <cylinder radius="0.02" length="0.0075"/>
+      </geometry>
+    </collision>
+    <inertial>
+      <mass value="${caster_mass}"/>
+      <inertia
+        ixx="${caster_ixx}" ixy="0.0" ixz="0.0"
+        iyy="${caster_iyy}" iyz="0.0"
+        izz="${caster_izz}"/>
+    </inertial>
+  </link>
+  <!-- Fixed, not a real swivel joint - the caster contributes no drive DOF
+       either way, and a fixed joint + near-zero friction contactMaterial
+       (see fix_proto.py/simulation.wbt's "caster_material") is the simplest
+       model that lets it slide freely as the diff-drive wheels steer. -->
+  <joint name="${prefix}caster_wheel_joint" type="fixed">
+    <parent link="${prefix}base_link"/>
+    <child link="${prefix}caster_wheel_link"/>
+    <origin xyz="${caster_x_offset} 0 ${caster_z_offset}" rpy="0 0 0"/>
+  </joint>
+  <!-- mu1/mu2 here are the Gazebo-path equivalent of the Webots
+       "caster_material" ContactProperties (simulation.wbt) - harmless
+       no-op under Webots, kept for RViz/Gazebo portability consistent with
+       how wheel.urdf.xacro's <gazebo> friction tags are handled. -->
+  <gazebo reference="${prefix}caster_wheel_link">
+    <mu1>0.001</mu1>
+    <mu2>0.001</mu2>
+  </gazebo>
 </xacro:macro>
 </robot>

File: src/amr_description/urdf/mech/wheel.urdf.xacro (robot description, xacro)
@@ -1,20 +1,43 @@
 <?xml version="1.0"?>
 <robot xmlns:xacro="http://www.ros.org/wiki/xacro">
+  <!-- Measured directly off rmp_bot's r_wheel_1.stl bounding box
+       (github.com/ravithakur-projects/ROS-Three-Wheeled-Robot-Navigation-Project):
+       X/Z extent ~65mm (diameter) -> radius 32.5mm, Y extent 25mm (width).
+       wheel_radius happens to numerically match this project's old mecanum
+       wheel radius exactly - coincidence, not reused from the old file.
+       wheel_mass is rmp_bot's own r_wheel_1 inertial mass (0.1182... kg). -->
   <xacro:property name="wheel_radius" value="0.0325" />
-  <xacro:property name="wheel_separation" value="0.169" />
-  <xacro:property name="wheel_width" value="0.03040" />
-  <xacro:property name="wheel_mass" value="0.15" />
-  <xacro:property name="wheel_xoff" value="0.08" />
-  <xacro:property name="wheel_yoff" value="-0.01" />
-  <!-- contact_material: "wheel_pos_45" for FL+RR (roller angle +45 deg),
-                          "wheel_neg_45" for FR+RL (roller angle -45 deg).
-       Injected as a Webots contactMaterial field on each wheel Solid
-       by fix_proto.py post-processing. No effect in Gazebo/RViz. -->
-  <xacro:macro name="wheel" params="prefix side x_reflect y_reflect contact_material">
+  <xacro:property name="wheel_width" value="0.025" />
+  <xacro:property name="wheel_mass" value="0.1182" />
+  <!-- rmp_bot joint origins: wheels at x=-0.05 (rear of base_link),
+       y=+-0.085 (track half-width) -> wheel_separation = 0.170m. -->
+  <xacro:property name="wheel_xoff" value="-0.05" />
+  <xacro:property name="wheel_separation" value="0.170" />
+  <!-- Plain differential-drive wheel - no contact_material split by
+       diagonal roller angle like the old mecanum macro had (both wheels
+       share the single "wheel_material" Webots ContactProperties entry,
+       see simulation.wbt/fix_proto.py), since these are ordinary wheels
+       with one rolling axis, not angled mecanum rollers. -->
+  <xacro:macro name="wheel" params="prefix side y_reflect">
     <link name="${prefix}${side}_wheel_link">
       <visual>
-        <origin xyz="0 0 0" rpy="1.5708 0 0"/>
+        <!-- NOT the old mecanum wheel's rpy="1.5708 0 0"/identity-origin
+             convention - that was for a differently-authored mesh. rmp_bot's
+             l_wheel_1.stl/r_wheel_1.stl raw vertices are already expressed
+             directly in base_link's own frame (a common quirk of the
+             Fusion360 URDF exporter: it cancels this out in its own xacro by
+             setting visual origin = -joint origin, e.g. r_wheel_1's joint is
+             at xyz="-0.05 -0.085 0.0325" and its visual origin is exactly
+             the negation, "0.05 0.085 -0.0325" - confirmed by reading their
+             xacro directly, not guessed). No rotation either: the mesh's
+             raw bounding box already has its thin 25mm dimension on Y (the
+             joint's own rotation axis), so it needs rpy 0 0 0, not a 90deg
+             flip. Reproducing that same cancellation here algebraically
+             (negative of this joint's own xyz) so the mesh recenters onto
+             wheel_link's local origin regardless of wheel_xoff/y_reflect. -->
+        <origin xyz="${-wheel_xoff} ${-y_reflect*(wheel_separation/2)} ${-wheel_radius}" rpy="0 0 0"/>
         <geometry>
-          <mesh filename="package://amr_description/meshes/${side}_wheel.stl"/>
+          <!-- rmp_bot's STLs are raw CAD exports in millimeters. -->
+          <mesh filename="package://amr_description/meshes/${side}_wheel.stl" scale="0.001 0.001 0.001"/>
         </geometry>
         <material name="dark_gray">
@@ -41,5 +64,5 @@
       <parent link="${prefix}base_link"/>
       <child link="${prefix}${side}_wheel_link"/>
-      <origin xyz="${x_reflect*wheel_xoff} ${y_reflect*(wheel_separation/2+wheel_yoff)} ${-wheel_radius}" rpy="0 0 0"/>
+      <origin xyz="${wheel_xoff} ${y_reflect*(wheel_separation/2)} ${wheel_radius}" rpy="0 0 0"/>
       <dynamics damping="0.01" friction="0.01"/>
       <limit effort="30.0" velocity="15.0"/>

File: src/amr_description/urdf/robots/amr.urdf.xacro (robot description, xacro)
@@ -14,26 +14,10 @@
     <xacro:wheel
       prefix="$(arg prefix)"
-      side="front_left"
-      x_reflect="1"
-      y_reflect="1"
-      contact_material="wheel_pos_45"/>
+      side="left"
+      y_reflect="1"/>
     <xacro:wheel
       prefix="$(arg prefix)"
-      side="front_right"
-      x_reflect="1"
-      y_reflect="-1"
-      contact_material="wheel_neg_45"/>
-    <xacro:wheel
-      prefix="$(arg prefix)"
-      side="rear_left"
-      x_reflect="-1"
-      y_reflect="1"
-      contact_material="wheel_neg_45"/>
-    <xacro:wheel
-      prefix="$(arg prefix)"
-      side="rear_right"
-      x_reflect="-1"
-      y_reflect="-1"
-      contact_material="wheel_pos_45"/>
+      side="right"
+      y_reflect="-1"/>
     <xacro:camera
       prefix="$(arg prefix)"
@@ -41,18 +25,20 @@
       xyz_offset="0.105 0 0.05"
       rpy_offset="0 0 0"/>
-    <!-- z=0.22: chassis.stl's own measured top is z=0.1905 (see
-         base.urdf.xacro's bbox comment). The previous xyz_offset (0.0825)
-         put the lidar's own mesh spanning roughly z=[0.062,0.101] -
-         entirely inside the chassis's 0.0540..0.1905 height range (measured
-         directly from lidar.stl + chassis.stl), so every one of its 360
-         rays hit the inside of its own chassis shell within centimeters
-         (well under minRange 0.1) and reported no return in every
-         direction, regardless of the room's actual wall distances. This
-         raises it clear of the chassis roof with a small margin. -->
+    <!-- Originally z=0.22, sized against the old 280x220x150mm mecanum
+         chassis (top at z=0.1905) - a 0.0295m clearance margin above the
+         chassis roof to clear a self-collision blind spot (see
+         decisions-and-gotchas.md). Left unchanged when the 2WD+caster
+         transition first landed, which left the lidar visibly floating
+         with a large gap above the new, much shorter chassis (top at
+         z=0.1175, see base.urdf.xacro) - confirmed visually in Webots/RViz.
+         Recomputed here with the SAME 0.0295m margin against the new
+         chassis top (0.1175 + 0.0295 = 0.1470, rounded to 0.15) rather than
+         reusing the old absolute height, closing the gap while keeping the
+         original design intent (small positive clearance, not flush). -->
     <xacro:lidar
       prefix="$(arg prefix)"
       parent="base_link"
       frame_id="laser_frame"
-      xyz_offset="0 0 0.22"
+      xyz_offset="0 0 0.15"
       rpy_offset="0 0 0"
       mesh_xyz_offset="0 0 0"
